Commit message: movement update & memory/spch

File: robot/dummy_lamp_5dof.urdf (robot description, URDF)
Before this commit: robot dummy_character_lamp_5dof, 10 links, 9 joints
Links:
- link lamp_head_link: geometry collision cylinder length=0.160 radius=0.110; visual cylinder length=0.006 radius=0.090
